File: Hardware/mini-vehiculo-exploracion-pcb/electrical.kicad_sch (KiCad schematic)
At the start: 21 parts, among them IC2 TPS564257DRLR

Commit message: cambio convertidor 3,3V a 5V
Parts:
- L1: value 3,3u -> 4,7u
- R16: value 45,3k -> 220k
- R17: value 10k -> 30k
Other:
- moved on the sheet: C19, C20, IC?
Changed lines of the file:
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@@
 		(exclude_from_sim no)
 		(at 30.48 19.05 0)
-		(size 168.91 60.96)
+		(size 179.07 60.96)
 		(margins 0.9525 0.9525 0.9525 0.9525)
 		(stroke
@@
 	(text_box "LDO 5V a 3,3V"
 		(exclude_from_sim no)
-		(at 200.66 20.32 0)
-		(size 67.31 52.07)
+		(at 212.09 20.32 0)
+		(size 69.85 41.91)
 		(margins 0.9525 0.9525 0.9525 0.9525)
 		(stroke
@@
 	)
 	(junction
-		(at 233.68 64.77)
+		(at 243.84 55.88)
 		(diameter 0)
 		(color 0 0 0 0)
@@
 	)
 	(junction
-		(at 213.36 41.91)
+		(at 223.52 33.02)
 		(diameter 0)
 		(color 0 0 0 0)
@@
 	)
 	(junction
-		(at 215.9 64.77)
+		(at 226.06 55.88)
 		(diameter 0)
 		(color 0 0 0 0)
@@
 	(wire
 		(pts
-			(xy 248.92 44.45) (xy 259.08 44.45)
+			(xy 259.08 35.56) (xy 269.24 35.56)
 		)
 		(stroke
@@
 	(wire
 		(pts
-			(xy 208.28 41.91) (xy 213.36 41.91)
+			(xy 218.44 33.02) (xy 223.52 33.02)
 		)
 		(stroke
@@
 	(wire
 		(pts
-			(xy 213.36 41.91) (xy 218.44 41.91)
+			(xy 223.52 33.02) (xy 228.6 33.02)
 		)
 		(stroke
@@
 	(wire
 		(pts
-			(xy 218.44 46.99) (xy 213.36 46.99)
+			(xy 228.6 38.1) (xy 223.52 38.1)
 		)
 		(stroke
@@
 	(wire
 		(pts
-			(xy 215.9 44.45) (xy 215.9 64.77)
+			(xy 226.06 35.56) (xy 226.06 55.88)
 		)
 		(stroke
@@
 	(wire
 		(pts
-			(xy 215.9 64.77) (xy 233.68 64.77)
-		)
-		(stroke
-			(width 0)
-			(type default)
-		)
-	)
-	(wire
-		(pts
-			(xy 213.36 46.99) (xy 213.36 41.91)
+			(xy 226.06 55.88) (xy 243.84 55.88)
+		)
+		(stroke
+			(width 0)
+			(type default)
+		)
+	)
+	(wire
+		(pts
+			(xy 223.52 38.1) (xy 223.52 33.02)
 		)
 		(stroke
@@
 	(wire
 		(pts
-			(xy 218.44 44.45) (xy 215.9 44.45)
+			(xy 228.6 35.56) (xy 226.06 35.56)
 		)
 		(stroke
@@
 	(wire
 		(pts
-			(xy 233.68 64.77) (xy 259.08 64.77)
+			(xy 243.84 55.88) (xy 269.24 55.88)
 		)
 		(stroke
@@
 	(wire
 		(pts
-			(xy 208.28 41.91) (xy 208.28 50.8)
+			(xy 218.44 33.02) (xy 218.44 41.91)
 		)
 		(stroke
@@
 	(wire
 		(pts
-			(xy 259.08 59.69) (xy 259.08 64.77)
+			(xy 269.24 50.8) (xy 269.24 55.88)
 		)
 		(stroke
@@
 	(wire
 		(pts
-			(xy 208.28 58.42) (xy 208.28 64.77)
+			(xy 218.44 49.53) (xy 218.44 55.88)
 		)
 		(stroke
@@
 	(wire
 		(pts
-			(xy 208.28 64.77) (xy 215.9 64.77)
-		)
-		(stroke
-			(width 0)
-			(type default)
-		)
-	)
-	(wire
-		(pts
-			(xy 259.08 44.45) (xy 259.08 52.07)
+			(xy 218.44 55.88) (xy 226.06 55.88)
+		)
+		(stroke
+			(width 0)
+			(type default)
+		)
+	)
+	(wire
+		(pts
+			(xy 269.24 35.56) (xy 269.24 43.18)
 		)
 		(stroke
@@
 	)
 	(label "V_IN"
-		(at 208.28 41.91 0)
+		(at 218.44 33.02 0)
 		(effects
 			(font
@@
 	)
 	(label "V_OUT"
-		(at 259.08 44.45 0)
+		(at 269.24 35.56 0)
 		(effects
 			(font
@@
 	(symbol
 		(lib_id "power:GND")
-		(at 233.68 64.77 0)
+		(at 243.84 55.88 0)
 		(unit 1)
 		(exclude_from_sim no)
@@
 		(fields_autoplaced yes)
 		(property "Reference" "#PWR022"
-			(at 233.68 71.12 0)
+			(at 243.84 62.23 0)
 			(effects
 				(font
@@
 		)
 		(property "Value" "GND"
-			(at 233.68 69.85 0)
+			(at 243.84 60.96 0)
 			(effects
 				(font
@@
 		)
 		(property "Footprint" ""
-			(at 233.68 64.77 0)
+			(at 243.84 55.88 0)
 			(effects
 				(font
@@
 		)
 		(property "Datasheet" ""
-			(at 233.68 64.77 0)
+			(at 243.84 55.88 0)
 			(effects
 				(font
@@
 		)
 		(property "Description" "Power symbol creates a global label with name \"GND\" , ground"
-			(at 233.68 64.77 0)
+			(at 243.84 55.88 0)
 			(effects
 				(font
@@
 			)
 		)
-		(property "Value" "10k"
+		(property "Value" "30k"
 			(at 179.07 63.4999 0)
 			(effects
@@
 	(symbol
 		(lib_id "Device:C")
-		(at 208.28 54.61 0)
+		(at 218.44 45.72 0)
 		(unit 1)
 		(exclude_from_sim no)
@@
 		(dnp no)
 		(property "Reference" "C19"
-			(at 212.09 53.3399 0)
+			(at 222.25 44.4499 0)
 			(effects
 				(font
@@
 		)
 		(property "Value" "1u"
-			(at 212.09 55.8799 0)
+			(at 222.25 46.9899 0)
 			(effects
 				(font
@@
 		)
 		(property "Footprint" ""
-			(at 209.2452 58.42 0)
+			(at 219.4052 49.53 0)
 			(effects
 				(font
@@
 		)
 		(property "Datasheet" "~"
-			(at 208.28 54.61 0)
+			(at 218.44 45.72 0)
 			(effects
 				(font
@@
 		)
 		(property "Description" "Unpolarized capacitor"
-			(at 208.28 54.61 0)
+			(at 218.44 45.72 0)
 			(effects
 				(font
@@
 	(symbol
 		(lib_id "MAX8891EXK33_V+T:MAX8891EXK33_V+T")
-		(at 218.44 41.91 0)
+		(at 228.6 33.02 0)
 		(unit 1)
 		(exclude_from_sim no)
@@
 		(fields_autoplaced yes)
 		(property "Reference" "IC?"
-			(at 233.68 34.29 0)
+			(at 243.84 25.4 0)
 			(effects
 				(font
@@
 		)
 		(property "Value" "MAX8891EXK33_V+T"
-			(at 233.68 36.83 0)
+			(at 243.84 27.94 0)
 			(effects
 				(font
@@
 		)
 		(property "Footprint" "SOT65P210X110-5N"
-			(at 245.11 136.83 0)
+			(at 255.27 127.94 0)
 			(effects
 				(font
@@
 		)
 		(property "Datasheet" "https://datasheets.maximintegrated.com/en/ds/MAX8891-MAX8892.pdf"
-			(at 245.11 236.83 0)
+			(at 255.27 227.94 0)
 			(effects
 				(font
@@
 		)
 		(property "Description" "IC REG LDO 3.3V 0.15A SC70-6"
-			(at 218.44 41.91 0)
+			(at 228.6 33.02 0)
 			(effects
 				(font
@@
 		)
 		(property "Height" "1.1"
-			(at 245.11 436.83 0)
+			(at 255.27 427.94 0)
 			(effects
 				(font
@@
 		)
 		(property "Mouser Part Number" ""
-			(at 245.11 536.83 0)
+			(at 255.27 527.94 0)
 			(effects
 				(font
@@
 		)
 		(property "Mouser Price/Stock" ""
-			(at 245.11 636.83 0)
+			(at 255.27 627.94 0)
 			(effects
 				(font
@@
 		)
 		(property "Manufacturer_Name" "Analog Devices"
-			(at 245.11 736.83 0)
+			(at 255.27 727.94 0)
 			(effects
 				(font
@@
 		)
 		(property "Manufacturer_Part_Number" "MAX8891EXK33/V+T"
-			(at 245.11 836.83 0)
+			(at 255.27 827.94 0)
 			(effects
 				(font
@@
 			)
 		)
-		(property "Value" "45,3k"
+		(property "Value" "220k"
 			(at 179.07 48.2599 0)
 			(effects
@@
 			)
 		)
-		(property "Value" "3,3u"
+		(property "Value" "4,7u"
 			(at 154.94 35.56 90)
 			(effects
@@
 	(symbol
 		(lib_id "Device:C")
-		(at 259.08 55.88 0)
+		(at 269.24 46.99 0)
 		(unit 1)
 		(exclude_from_sim no)
@@
 		(fields_autoplaced yes)
 		(property "Reference" "C20"
-			(at 262.89 54.6099 0)
+			(at 273.05 45.7199 0)
 			(effects
 				(font
@@
 		)
 		(property "Value" "1u"
-			(at 262.89 57.1499 0)
+			(at 273.05 48.2599 0)
 			(effects
 				(font
@@
 		)
 		(property "Footprint" ""
-			(at 260.0452 59.69 0)
+			(at 270.2052 50.8 0)
 			(effects
 				(font
@@
 		)
 		(property "Datasheet" "~"
-			(at 259.08 55.88 0)
+			(at 269.24 46.99 0)
 			(effects
 				(font
@@
 		)
 		(property "Description" "Unpolarized capacitor"
-			(at 259.08 55.88 0)
-			(effects
-				(font
+			(at 269.24 46.99 0)
+			(effects
+				(font

Commit message: actualizacion labels pcb de control
Parts:
- removed D?: D_Schottky, symbol Device:D_Schottky
- added D5: PMEG040V030EPE-QZ, PMEG040V030EPEQZ, symbol PMEG040V030EPE-QZ:PMEG040V030EPE-QZ
Connections:
- net V_BAT: now also C16.1, C17.1, C18.1, L1.2, R15.2, R16.1
- net V_BUS renamed +5V
- net +5V: now also D5.1 (A_1), D5.2 (A_2)
- net V_IN renamed 12V
- net 12V: no longer C19.1, IC?.1 (IN), IC?.3 (~{SHDN})
- removed net V_OUT: C16.1, C17.1, C18.1, C20.1, IC?.5 (OUT), L1.2, Q?.4 (S), R15.2, R16.1
- new net +3.3V: C20.1, IC?.5 (OUT)
- new net V_SELEC: C19.1, D5.3 (K), IC?.1 (IN), IC?.3 (~{SHDN}), Q?.4 (S)
