File: Hardware/mini-vehiculo-exploracion-pcb/electrical.kicad_sch (KiCad schematic)
At the start: 16 parts, among them IC3 MAX8891EXK33_V+T, Q1 SI1467DH-T1-BE3, U4 TPS561208DDCR

Commit message: Reorder
Other:
- title: (none) -> Vehiculo de exploracion a escala
Changed lines of the file:
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@@
 	(generator_version "9.0")
 	(paper "A4")
+	(title_block
+		(title "Vehiculo de exploracion a escala")
+		(date "2026-03-28")
+		(rev "1.0")
+	)
 	(text_box "Entrada 12V Bateria\n"
 		(exclude_from_sim no)
