File: Hardware/mini-vehiculo-exploracion-pcb/mini-vehiculo-exploracion-pcb.kicad_pcb (KiCad board)
At the start: 2 copper layers, 0 parts

Commit message: innit pcb
Parts:
- added C1: 0.1uF, Capacitor_SMD:C_0805_2012Metric_Pad1.18x1.45mm_HandSolder, F.Cu at (99.0, 78.0)
- added C10: 0.1uF, Capacitor_SMD:C_0805_2012Metric_Pad1.18x1.45mm_HandSolder, F.Cu at (153.0, 51.5)
- added C11: 0.1uF, Capacitor_SMD:C_0805_2012Metric_Pad1.18x1.45mm_HandSolder, F.Cu at (202.0, 44.5)
- added C12: 0.1uF, Capacitor_SMD:C_0805_2012Metric_Pad1.18x1.45mm_HandSolder, F.Cu at (163.5, 67.0)
- added C13: 1uF, Capacitor_SMD:C_0805_2012Metric_Pad1.18x1.45mm_HandSolder, F.Cu at (196.8, 60.5)
- added C14: 100n, Capacitor_SMD:C_0805_2012Metric_Pad1.18x1.45mm_HandSolder, F.Cu at (154.9, 79.2)
- added C15: 47u, Capacitor_SMD:C_0805_2012Metric_Pad1.18x1.45mm_HandSolder, F.Cu at (142.0, 76.5)
- added C16: 10u, Capacitor_SMD:C_0805_2012Metric_Pad1.18x1.45mm_HandSolder, F.Cu at (154.9, 85.3)
- added C17: 10uF, Capacitor_SMD:C_0805_2012Metric_Pad1.18x1.45mm_HandSolder, F.Cu at (157.0, 125.0)
- added C18: 4.7u, Capacitor_SMD:C_0805_2012Metric_Pad1.18x1.45mm_HandSolder, F.Cu at (160.0, 118.5)
- added C19: 1u, Capacitor_SMD:C_0805_2012Metric_Pad1.18x1.45mm_HandSolder, F.Cu at (136.5, 66.5)
- added C2: 0.1uF, Capacitor_SMD:C_0805_2012Metric_Pad1.18x1.45mm_HandSolder, F.Cu at (139.5, 96.5)
- added C20: 1u, Capacitor_SMD:C_0805_2012Metric_Pad1.18x1.45mm_HandSolder, F.Cu at (154.9, 91.3)
- added C21: 10uF, Capacitor_SMD:C_0805_2012Metric_Pad1.18x1.45mm_HandSolder, F.Cu at (153.0, 113.5)
- added C22: 200nF, Capacitor_SMD:C_0805_2012Metric_Pad1.18x1.45mm_HandSolder, F.Cu at (174.0, 114.5)
- added C3: 0.1uF, Capacitor_SMD:C_0805_2012Metric_Pad1.18x1.45mm_HandSolder, F.Cu at (112.0, 119.0)
- added C4: 22pF, Capacitor_SMD:C_0805_2012Metric_Pad1.18x1.45mm_HandSolder, F.Cu at (92.5, 117.5)
- added C5: 22pF, Capacitor_SMD:C_0805_2012Metric_Pad1.18x1.45mm_HandSolder, F.Cu at (92.5, 127.0)
- added C6: 100n, Capacitor_SMD:C_0805_2012Metric_Pad1.18x1.45mm_HandSolder, F.Cu at (139.5, 108.5)
- added C7: 100n, Capacitor_SMD:C_0805_2012Metric_Pad1.18x1.45mm_HandSolder, F.Cu at (139.5, 111.5)
- added C8: 1uF, Capacitor_SMD:C_0805_2012Metric_Pad1.18x1.45mm_HandSolder, F.Cu at (196.5, 30.5)
- added C9: 22uF, Capacitor_SMD:C_0805_2012Metric_Pad1.18x1.45mm_HandSolder, F.Cu at (161.0, 51.5)
- added CR1: USBLC6-2SC6, USB_PROTECTION_SOT23-6L_STM:SOT23-6L_STM, F.Cu at (219.5, 70.0)
- added D1: D_Schottky, USB_diode_SD1206S040S1R0:SD1206_AVX, F.Cu at (174.8, 67.0)
- added D2: 82350120560, Diode_82350120560:CR_50120560_WRE-M, F.Cu at (196.9, 65.5)
- added D3: PTVS13VP1UTP-QX, PTVS13VP1UTP-QX:SODFL4725X110N, F.Cu at (207.9, 126.0)
- added D4: PMEG040V030EPE-QZ, PMEG040V030EPE-QZ:PMEG040V030EPEQZ, F.Cu at (132.0, 50.1)
- added D5: PMEG040V030EPE-QZ, PMEG040V030EPE-QZ:PMEG040V030EPEQZ, F.Cu at (129.5, 67.6)
- added D6: GREEN, LED_SMD:LED_0805_2012Metric, F.Cu at (175.6, 45.0)
- added F1: Polyfuse, USB_fuse_C1Q-1:C1_BEL, F.Cu at (184.5, 46.0)
- added F3: SMD100F-2018-2, SMD100F-2018-2:SMD030F20182, F.Cu at (118.5, 53.0)
- added FB1: BLM21PG221SN1D, USB_FerriteBead_IND_BLM21_MUR:IND_BLM21_MUR, F.Cu at (186.5, 51.0)
- added IC1: BME690, BME690:BME690, F.Cu at (108.2, 77.4)
- added IC3: MAX8891EXK33_V+T, MAX8891EXK33_V+T:SOT65P210X110-5N, F.Cu at (134.0, 74.0)
- added J1: Cámara, ArducamMINIOV2640:ArducamMINIOV2640, F.Cu at (228.1, 84.5)
- added J2: USB_C_Receptacle_USB2.0_16P, USB_UJ20-C-H-G-SMT-P16-TR:SAMESKY_UJ20-C-H-G-SMT-P16-TR, F.Cu at (218.0, 61.0)
- added J3: Drivers_Conn_1x8, Connector_PinSocket_2.54mm:PinSocket_1x08_P2.54mm_Vertical, F.Cu at (209.5, 67.5)
- added J4: Drivers_Conn_1x4, Connector_PinSocket_2.54mm:PinSocket_1x04_P2.54mm_Vertical, F.Cu at (264.5, 83.7)
- added J5: Aux_Conn_1x4, Connector_PinSocket_2.54mm:PinSocket_1x04_P2.54mm_Vertical, F.Cu at (264.5, 72.2)
- added J6: RC_Conn_1x4, Connector_PinSocket_2.54mm:PinSocket_1x04_P2.54mm_Vertical, F.Cu at (264.5, 60.7)
- added J7: Battery_Terminal_01x02, TerminalBlock:TerminalBlock_Xinya_XY308-2.54-2P_1x02_P2.54mm_Horizontal, F.Cu at (147.0, 29.5)
- added L2: MLP2520S4R7MT0S1, MLP2520S4R7MT0S1:INDC2520X100N, F.Cu at (160.5, 79.5)
- added Q1: SI1467DH-T1-BE3, SI1467DH-T1-BE3:SOT65P210X110-6N, F.Cu at (143.1, 70.5)
- added R1: 4.7k, Resistor_SMD:R_0805_2012Metric_Pad1.20x1.40mm_HandSolder, F.Cu at (108.5, 68.5)
- added R10: 5.1K, Resistor_SMD:R_0805_2012Metric_Pad1.20x1.40mm_HandSolder, F.Cu at (189.0, 81.0)
- added R11: 5.1K, Resistor_SMD:R_0805_2012Metric_Pad1.20x1.40mm_HandSolder, F.Cu at (195.5, 82.5)
- added R12: 10K, Resistor_SMD:R_0805_2012Metric_Pad1.20x1.40mm_HandSolder, F.Cu at (204.4, 60.5)
- added R13: 56,2k, Resistor_SMD:R_0805_2012Metric_Pad1.20x1.40mm_HandSolder, F.Cu at (162.5, 75.0)
- added R14: 10k, Resistor_SMD:R_0805_2012Metric_Pad1.20x1.40mm_HandSolder, F.Cu at (167.5, 75.0)
- added R15: 10k, Resistor_SMD:R_0805_2012Metric_Pad1.20x1.40mm_HandSolder, F.Cu at (148.5, 103.0)
- added R16: 18k, Resistor_SMD:R_0805_2012Metric_Pad1.20x1.40mm_HandSolder, F.Cu at (148.0, 108.0)
- added R17: 20k, Resistor_SMD:R_0805_2012Metric_Pad1.20x1.40mm_HandSolder, F.Cu at (148.0, 113.5)
- added R18: 1k, Resistor_SMD:R_0805_2012Metric_Pad1.20x1.40mm_HandSolder, F.Cu at (175.5, 50.0)
- added R19: 10k, Resistor_SMD:R_0805_2012Metric_Pad1.20x1.40mm_HandSolder, F.Cu at (174.5, 63.0)
- added R2: 4.7k, Resistor_SMD:R_0805_2012Metric_Pad1.20x1.40mm_HandSolder, F.Cu at (108.0, 85.0)
- added R20: 2k, Resistor_SMD:R_0805_2012Metric_Pad1.20x1.40mm_HandSolder, F.Cu at (148.5, 118.5)
- added R21: 2.7k, Resistor_SMD:R_0805_2012Metric_Pad1.20x1.40mm_HandSolder, F.Cu at (154.9, 118.6)
- added R3: 10K, Resistor_SMD:R_0805_2012Metric_Pad1.20x1.40mm_HandSolder, F.Cu at (202.0, 34.5)
- added R4: 65k, Resistor_SMD:R_0805_2012Metric_Pad1.20x1.40mm_HandSolder, F.Cu at (150.0, 98.0)
- added R5: 2.2k, Resistor_SMD:R_0805_2012Metric_Pad1.20x1.40mm_HandSolder, F.Cu at (119.5, 130.0)
- added R6: 2.2k, Resistor_SMD:R_0805_2012Metric_Pad1.20x1.40mm_HandSolder, F.Cu at (116.0, 137.5)
- added R7: 10k, Resistor_SMD:R_0805_2012Metric_Pad1.20x1.40mm_HandSolder, F.Cu at (117.0, 117.0)
- added R8: 2.2k, Resistor_SMD:R_0805_2012Metric_Pad1.20x1.40mm_HandSolder, F.Cu at (106.0, 135.5)
- added R9: 2.2k, Resistor_SMD:R_0805_2012Metric_Pad1.20x1.40mm_HandSolder, F.Cu at (119.5, 123.5)
- added S1: B3FS-1010, B3FS-1010:B3FS-1000P, F.Cu at (193.5, 37.0)
- added S2: B3FS-1010, B3FS-1010:B3FS-1000P, F.Cu at (187.5, 60.5)
- added TP1: Bat_div, TestPoint:TestPoint_Pad_1.5x1.5mm, F.Cu at (176.5, 126.0)
- added TP2: OP1_Out, TestPoint:TestPoint_Pad_1.5x1.5mm, F.Cu at (147.0, 124.5)
- added TP3: OP2_Out, TestPoint:TestPoint_Pad_1.5x1.5mm, F.Cu at (163.8, 122.9)
- added U1: BNO086, BNO086:BNO086, F.Cu at (113.5, 128.5)
- added U2: ESP32-S3-WROOM-1, RF_Module:ESP32-S3-WROOM-1, F.Cu at (237.0, 65.1)
- added U3: LM358, LM358AN_NOPB:DIP794W53P254L959H508Q8N, F.Cu at (186.0, 115.5)
- added U4: TPS561208DDCR, TPS561208DDCR:SOT95P280X110-6N, F.Cu at (194.8, 104.5)
- added Y1: 830003000, 830003000:830003000, F.Cu at (94.2, 122.3)
Routing:
- net Net-(U1-ENV_SCL): track 0.00 -> 7.97 mm
- net /RX_1: track 0.00 -> 7.83 mm
- net /XTAL_N: track 0.00 -> 3.70 mm
- net /XTAL_P: track 0.00 -> 3.50 mm
