File: Hardware/mini-vehiculo-exploracion-pcb/mini-vehiculo-exploracion-pcb.kicad_pcb (KiCad board)
At the start: 2 copper layers, 74 parts, among them IC1 BME690, IC3 MAX8891EXK33_V+T, J1 Cámara, J2 USB_C_Receptacle_USB2.0_16P, J3 Drivers_Conn_1x8, J4 Drivers_Conn_1x4, J5 Aux_Conn_1x4, J6 RC_Conn_1x4, J7 Battery_Terminal_01x02, Q1 SI1467DH-T1-BE3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

Commit message: Add netclassses, mounting holes and terminal block
Parts:
- J1: value Cámara -> ArducamMINIOV2640
- J7: footprint TerminalBlock:TerminalBlock_Xinya_XY308-2.54-2P_1x02_P2.54mm_Horizontal -> TerminalBlock_Phoenix:TerminalBlock_Phoenix_MPT-0,5-2-2.54_1x02_P2.54mm_Horizontal
Connections:
- J3 pad 4: unconnected-(J3-Pin_4-Pad4) -> /SERVO_CRL

Commit message: Update pcb from schematic
Parts:
- added H1: MountingHole_Pad, MountingHole:MountingHole_3.2mm_M3_Pad_Via, F.Cu at (64.4, 74.8)
- added H2: MountingHole_Pad, MountingHole:MountingHole_3.2mm_M3_Pad_Via, F.Cu at (64.4, 82.8)
- added H3: MountingHole_Pad, MountingHole:MountingHole_3.2mm_M3_Pad_Via, F.Cu at (64.4, 90.7)
- added H4: MountingHole_Pad, MountingHole:MountingHole_3.2mm_M3_Pad_Via, F.Cu at (64.4, 98.7)
- added J4: Conn_01x02_Pin, Connector_PinSocket_2.54mm:PinSocket_1x02_P2.54mm_Vertical, F.Cu at (70.7, 73.2)

Commit message: continue pcb
Parts:
- removed the J4 at (264.5, 83.7)
- added C23: 0.1uF, Capacitor_SMD:C_0805_2012Metric_Pad1.18x1.45mm_HandSolder, F.Cu at (98.5, 90.0)
- added C24: 0.1uF, Capacitor_SMD:C_0805_2012Metric_Pad1.18x1.45mm_HandSolder, F.Cu at (95.0, 96.5)
- added IC2: TXU0104PWR, TXU0104PWR:SOP65P640X120-14N, F.Cu at (88.0, 83.0)
- added J8: SERVO, Connector_PinSocket_2.54mm:PinSocket_1x03_P2.54mm_Vertical, F.Cu at (106.0, 80.0)
- J4: value Conn_01x02_Pin -> MOTORES
- PLACA DRIVERS: renamed from J3
- moved CR1 182.3 mm to (41.0, 33.0), turned to -90 degrees
- moved J2 180.9 mm to (41.0, 23.5)
- moved U2 177.0 mm to (64.0, 27.6)
- moved J1 175.1 mm to (55.1, 57.5)
- moved R11 167.5 mm to (35.5, 33.0), turned to 90 degrees
- moved AUX 158.9 mm to (106.0, 61.4)
- moved RC 158.9 mm to (106.0, 49.9)
- moved D3 151.3 mm to (63.5, 81.0)
- moved R10 149.4 mm to (47.5, 33.0), turned to 90 degrees
- moved PLACA DRIVERS 139.5 mm to (76.1, 108.5), turned to 90 degrees
- moved J7 137.3 mm to (33.0, 106.0)
- moved C2 125.2 mm to (25.0, 45.9), turned to 90 degrees
- moved U3 122.0 mm to (95.7, 33.5), turned to 90 degrees
- moved U4 120.6 mm to (74.8, 92.0)
- moved R14 118.4 mm to (50.0, 89.5), turned to 90 degrees
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- renumbered J5 to AUX, IC1 to BME690, J6 to RC
Connections:
- PLACA DRIVERS pad 4: /SERVO_CRL -> unconnected-(J3-Pin_4-Pad4)
Routing:
- net /XTAL_N: track 3.70 -> 28.0 mm
- net /XTAL_P: track 3.50 -> 25.8 mm
- net ADC_BAT: track 0.00 -> 17.7 mm
- net /Battery_sensor/OP1_OUT: track 0.00 -> 16.1 mm
- net Net-(U1-ENV_SCL): track 7.97 -> 2.88 mm
- net /RX_1: track 7.83 -> 3.60 mm
- net +3.3V: track 0.00 -> 3.52 mm
- net Net-(U1-ENV_SDA): track 0.00 -> 3.19 mm
- net /TX_1: track 0.00 -> 3.00 mm
- net Net-(U1-CAP): track 0.00 -> 2.88 mm
- added copper zone on B.Cu, net GND

Commit message: change pcb2
Parts:
- D6: value GREEN -> ON
- J1: value ArducamMINIOV2640 -> Cámara
- moved R3 164.2 mm to (95.0, 66.0), turned to -90 degrees
- moved C11 159.0 mm to (98.5, 66.0), turned to -90 degrees
- moved EN 153.6 mm to (98.0, 71.5)
- moved C8 152.9 mm to (102.0, 66.0), turned to -90 degrees
- moved FB1 139.3 mm to (101.0, 53.3), turned to 90 degrees
- moved F1 134.6 mm to (104.0, 53.9), turned to -90 degrees
- moved D1 131.5 mm to (97.6, 53.9), turned to 90 degrees
- moved C9 125.4 mm to (91.5, 72.8), turned to -90 degrees
- moved R19 123.3 mm to (106.9, 82.5), turned to 90 degrees
- moved C10 116.8 mm to (91.5, 68.5), turned to -90 degrees
- moved C12 113.8 mm to (103.5, 60.5), turned to 90 degrees
- moved R12 110.0 mm to (153.5, 92.4), turned to 90 degrees
- moved D2 108.0 mm to (146.5, 92.3), turned to -90 degrees
- moved C13 106.1 mm to (150.0, 92.4), turned to -90 degrees
- moved C20 103.2 mm to (106.8, 73.0), turned to -90 degrees
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- renumbered J7 to BATERÍA, U1 to BNO086, S2 to BOOT, S1 to EN, IC2 to TR
Routing:
- net +3.3V: track 3.52 -> 54.7 mm
- net V_SELEC: track 0.00 -> 22.6 mm
- net /SERVO_CRL: track 0.00 -> 22.1 mm
- net Net-(U4-VFB): track 0.00 -> 18.8 mm
- net Net-(D4-K): track 0.00 -> 17.3 mm
- net /Battery_sensor/OP1_OUT: track 16.1 -> 33.0 mm
- net ENT_BAT: track 0.00 -> 16.7 mm
- net V_BAT: track 0.00 -> 16.2 mm
- net Net-(R15-Pad2): track 0.00 -> 15.8 mm
- net /M1_nFAULT: track 0.00 -> 15.1 mm
- net /M2_nFAULT: track 0.00 -> 12.4 mm
- net V_BUS: track 0.00 -> 11.9 mm
- net Net-(C22-Pad1): track 0.00 -> 10.8 mm
- net /SERVO_SAL: track 0.00 -> 10.4 mm
- net ESP_IO0: track 0.00 -> 9.36 mm
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
Commit message: update pcb3
Parts:
- removed AUX: Aux_Conn_1x4, Connector_PinSocket_2.54mm:PinSocket_1x04_P2.54mm_Vertical
- removed J2: USB_C_Receptacle_USB2.0_16P, USB_UJ20-C-H-G-SMT-P16-TR:SAMESKY_UJ20-C-H-G-SMT-P16-TR
- removed PLACA DRIVERS: Drivers_Conn_1x8, Connector_PinSocket_2.54mm:PinSocket_1x08_P2.54mm_Vertical
- added AUX1: AUX, Connector_PinSocket_2.54mm:PinSocket_1x03_P2.54mm_Vertical, F.Cu at (146.2, 60.6)
- added DRIVERS_DER1: DRIVERS_DER, Connector_PinSocket_2.54mm:PinSocket_1x04_P2.54mm_Vertical, F.Cu at (142.5, 115.7)
- added DRIVERS_IZQ1: DRIVERS_IZQ, Connector_PinSocket_2.54mm:PinSocket_1x04_P2.54mm_Vertical, F.Cu at (121.4, 115.6)
- added J3: UJ20-C-H-G-SMT-5-P16-TR, USB_UJ20-C-H-G-SMT-P16-TR:UJ20CHGSMT5P16TR, F.Cu at (171.4, 102.5)
- J1: value Cámara -> CÁMARA
- RC1: renamed from RC; value RC_Conn_1x4 -> RC
- U2: footprint RF_Module:ESP32-S3-WROOM-1 -> ESP32-S3-WROOM-1-P3JLC:ESP32-S3-WROOM-1-P3JLC
- moved D1 79.4 mm to (157.1, 106.3), turned to -90 degrees
- moved FB1 75.4 mm to (154.1, 106.8), turned to -90 degrees
- moved C12 74.6 mm to (161.2, 107.9), turned to 0 degrees
- moved F1 70.4 mm to (151.1, 106.2), turned to 90 degrees
- moved R11 64.5 mm to (161.1, 97.2), turned to 180 degrees
- moved CR1 63.9 mm to (161.1, 100.8), turned to 180 degrees
- moved R10 63.1 mm to (161.1, 104.2), turned to 180 degrees
- moved D6 59.9 mm to (97.0, 87.1)
- moved R18 59.9 mm to (99.5, 87.0)
- moved BNO086 46.4 mm to (94.6, 74.8)
- moved C2 46.4 mm to (92.1, 65.2)
- moved R5 46.4 mm to (99.1, 76.0)
- moved R6 46.4 mm to (96.3, 81.2)
- moved R7 46.4 mm to (94.3, 69.2)
- moved R8 46.4 mm to (90.1, 78.0)
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- renumbered BATERÍA to BATERÍA1, BOOT to BOOT1, Y1 to CRISTAL1, J4 to MOTORES1, EN to S1, TR to TR1
Connections:
- C24 pad 1: V_SELEC -> V_BAT
- F1 pad 1: Net-(F1-Pad1) -> V_BUS
- J8 pad 2: V_SELEC -> V_BAT
- TR1 pad 14: V_SELEC -> V_BAT
- U2 pad 35: /PIN_AUX3 -> /ADC_BAT2
Routing:
- net GND: track 0.00 -> 544.9 mm, vias 0 -> 24
- net +3.3V: track 54.7 -> 350.0 mm, vias 0 -> 9
- net /M1_DISABLE: track 0.00 -> 179.9 mm, vias 0 -> 1
- net /M1_IN1: track 0.00 -> 149.7 mm, vias 0 -> 1
- net ENT_BAT: track 16.7 -> 166.3 mm
- net /M1_IN2: track 0.00 -> 138.3 mm, vias 0 -> 1
- net /M2_IN2: track 0.00 -> 122.1 mm, vias 0 -> 1
- net /M2_DISABLE: track 0.00 -> 110.0 mm, vias 0 -> 1
- net V_BAT: track 16.2 -> 123.0 mm
- net V_BUS: track 11.9 -> 116.8 mm
- net /ADC_BAT2: track 0.00 -> 95.8 mm, vias 0 -> 1
- net /M2_IN1: track 0.00 -> 87.8 mm, vias 0 -> 1
- net /BNO_INT: track 0.00 -> 76.8 mm
- net USB_D-: track 0.00 -> 70.5 mm
- net USB_D+: track 0.00 -> 66.3 mm
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- added copper zone on F.Cu, net GND
Other:
- board outline added: 92 x 79 mm
