File: Hardware/mini-vehiculo-exploracion-pcb/battery_sensor.kicad_sch (KiCad schematic)
At the start: 14 parts, among them U3 LM358

Commit message: adicion de bornera pcb drivers y organizacion de entrada
Parts:
- renumbered C21 to C18, C22 to C19, C17 to C20, C18 to C21, R15 to R10, R16 to R11, R17 to R12, R20 to R13, R21 to R14, R4 to R9, U3 to U4
Changed lines of the file:
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@@
 		(dnp no)
 		(fields_autoplaced yes)
-		(property "Reference" "C18"
+		(property "Reference" "C21"
 			(at 219.71 66.04 90)
 			(effects
@@
 			(project "drivers-mini-vehiculo-pcb"
 				(path "/7776e3ee-622a-4a3e-a213-279f6f5df2cb/09f4a7ab-b5f1-4ef7-9bc4-d2f318ad2ada"
-					(reference "C?")
+					(reference "C21")
 					(unit 1)
 				)
@@
 		(dnp no)
 		(fields_autoplaced yes)
-		(property "Reference" "C17"
+		(property "Reference" "C20"
 			(at 208.28 110.4899 0)
 			(effects
@@
 			(project "drivers-mini-vehiculo-pcb"
 				(path "/7776e3ee-622a-4a3e-a213-279f6f5df2cb/09f4a7ab-b5f1-4ef7-9bc4-d2f318ad2ada"
-					(reference "C?")
+					(reference "C20")
 					(unit 1)
 				)
@@
 		(dnp no)
 		(fields_autoplaced yes)
-		(property "Reference" "R15"
+		(property "Reference" "R10"
 			(at 57.15 110.4899 0)
 			(effects
@@
 			(project "drivers-mini-vehiculo-pcb"
 				(path "/7776e3ee-622a-4a3e-a213-279f6f5df2cb/09f4a7ab-b5f1-4ef7-9bc4-d2f318ad2ada"
-					(reference "R?")
+					(reference "R10")
 					(unit 1)
 				)
@@
 		(dnp no)
 		(fields_autoplaced yes)
-		(property "Reference" "R16"
+		(property "Reference" "R11"
 			(at 76.2 96.52 90)
 			(effects
@@
 			(project "drivers-mini-vehiculo-pcb"
 				(path "/7776e3ee-622a-4a3e-a213-279f6f5df2cb/09f4a7ab-b5f1-4ef7-9bc4-d2f318ad2ada"
-					(reference "R?")
+					(reference "R11")
 					(unit 1)
 				)
@@
 		(on_board yes)
 		(dnp no)
-		(property "Reference" "U3"
+		(property "Reference" "U4"
 			(at 218.44 107.95 0)
 			(effects
@@
 		(dnp no)
 		(fields_autoplaced yes)
-		(property "Reference" "#PWR027"
+		(property "Reference" "#PWR0103"
 			(at 111.76 127 0)
 			(effects
@@
 		(dnp no)
 		(fields_autoplaced yes)
-		(property "Reference" "U3"
+		(property "Reference" "U4"
 			(at 109.22 53.3399 0)
 			(effects
@@
 		(dnp no)
 		(fields_autoplaced yes)
-		(property "Reference" "C21"
+		(property "Reference" "C18"
 			(at 115.57 111.7599 0)
 			(effects
@@
 		(dnp no)
 		(fields_autoplaced yes)
-		(property "Reference" "#PWR029"
+		(property "Reference" "#PWR0101"
 			(at 204.47 125.73 0)
 			(effects
@@
 			(project "drivers-mini-vehiculo-pcb"
 				(path "/7776e3ee-622a-4a3e-a213-279f6f5df2cb/09f4a7ab-b5f1-4ef7-9bc4-d2f318ad2ada"
-					(reference "TP?")
+					(reference "TP2")
 					(unit 1)
 				)
@@
 		(dnp no)
 		(fields_autoplaced yes)
-		(property "Reference" "R20"
+		(property "Reference" "R13"
 			(at 180.34 93.98 90)
 			(effects
@@
 			(project "drivers-mini-vehiculo-pcb"
 				(path "/7776e3ee-622a-4a3e-a213-279f6f5df2cb/09f4a7ab-b5f1-4ef7-9bc4-d2f318ad2ada"
-					(reference "R?")
+					(reference "R13")
 					(unit 1)
 				)
@@
 		(dnp no)
 		(fields_autoplaced yes)
-		(property "Reference" "U3"
+		(property "Reference" "U4"
 			(at 130.81 90.17 0)
 			(effects
@@
 		(dnp no)
 		(fields_autoplaced yes)
-		(property "Reference" "#PWR026"
+		(property "Reference" "#PWR015"
 			(at 54.61 127 0)
 			(effects
@@
 		(dnp no)
 		(fields_autoplaced yes)
-		(property "Reference" "R4"
+		(property "Reference" "R9"
 			(at 57.15 90.1699 0)
 			(effects
@@
 		(dnp no)
 		(fields_autoplaced yes)
-		(property "Reference" "R17"
+		(property "Reference" "R12"
 			(at 99.06 96.52 90)
 			(effects
@@
 			(project "drivers-mini-vehiculo-pcb"
 				(path "/7776e3ee-622a-4a3e-a213-279f6f5df2cb/09f4a7ab-b5f1-4ef7-9bc4-d2f318ad2ada"
-					(reference "R?")
+					(reference "R12")
 					(unit 1)
 				)
@@
 			(project "drivers-mini-vehiculo-pcb"
 				(path "/7776e3ee-622a-4a3e-a213-279f6f5df2cb/09f4a7ab-b5f1-4ef7-9bc4-d2f318ad2ada"
-					(reference "TP?")
+					(reference "TP3")
 					(unit 1)
 				)
@@
 		(dnp no)
 		(fields_autoplaced yes)
-		(property "Reference" "R21"
+		(property "Reference" "R14"
 			(at 198.12 93.98 90)
 			(effects
@@
 			(project "drivers-mini-vehiculo-pcb"
 				(path "/7776e3ee-622a-4a3e-a213-279f6f5df2cb/09f4a7ab-b5f1-4ef7-9bc4-d2f318ad2ada"
-					(reference "R?")
+					(reference "R14")
 					(unit 1)
 				)
@@
 		(dnp no)
 		(fields_autoplaced yes)
-		(property "Reference" "#PWR028"
+		(property "Reference" "#PWR0102"
 			(at 107.95 71.12 0)
 			(effects
@@
 		(dnp no)
 		(fields_autoplaced yes)
-		(property "Reference" "C22"
+		(property "Reference" "C19"
 			(at 132.08 67.31 90)
 			(effects
