File: Hardware/mini-vehiculo-exploracion-pcb/battery_sensor.kicad_sch (KiCad schematic)
At the start: 14 parts, among them U3 LM358

Commit message: updated pcb drv
Parts:
- renumbered C21 to C18, C22 to C19, C24 to C20, C23 to C21, R20 to R10, R21 to R11, R22 to R12, R23 to R13, R24 to R14, R4 to R9, U3 to U4
Changed lines of the file:
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@@
 		(dnp no)
 		(fields_autoplaced yes)
-		(property "Reference" "R21"
+		(property "Reference" "R11"
 			(at 76.2 96.52 90)
 			(effects
@@
 				)
 			)
+			(project "mini-vehiculo-exploracion-pcb"
+				(path "/7776e3ee-622a-4a3e-a213-279f6f5df2cb/09f4a7ab-b5f1-4ef7-9bc4-d2f318ad2ada"
+					(reference "R11")
+					(unit 1)
+				)
+			)
 		)
 	)
@@
 		(dnp no)
 		(fields_autoplaced yes)
-		(property "Reference" "R22"
+		(property "Reference" "R12"
 			(at 99.06 96.52 90)
 			(effects
@@
 				(path "/3cb3b833-c38f-47b4-b7e9-f0e6337b7613/27757aec-ab0f-470c-ac2a-d85fc9232d35"
 					(reference "R22")
+					(unit 1)
+				)
+			)
+			(project "mini-vehiculo-exploracion-pcb"
+				(path "/7776e3ee-622a-4a3e-a213-279f6f5df2cb/09f4a7ab-b5f1-4ef7-9bc4-d2f318ad2ada"
+					(reference "R12")
 					(unit 1)
 				)
@@
 		(on_board yes)
 		(dnp no)
-		(property "Reference" "U3"
+		(property "Reference" "U4"
 			(at 218.44 107.95 0)
 			(effects
@@
 				)
 			)
+			(project ""
+				(path "/7776e3ee-622a-4a3e-a213-279f6f5df2cb/09f4a7ab-b5f1-4ef7-9bc4-d2f318ad2ada"
+					(reference "U4")
+					(unit 2)
+				)
+			)
 		)
 	)
@@
 		(dnp no)
 		(fields_autoplaced yes)
-		(property "Reference" "#PWR027"
+		(property "Reference" "#PWR017"
 			(at 111.76 127 0)
 			(effects
@@
 				(path "/3cb3b833-c38f-47b4-b7e9-f0e6337b7613/27757aec-ab0f-470c-ac2a-d85fc9232d35"
 					(reference "#PWR027")
+					(unit 1)
+				)
+			)
+			(project "mini-vehiculo-exploracion-pcb"
+				(path "/7776e3ee-622a-4a3e-a213-279f6f5df2cb/09f4a7ab-b5f1-4ef7-9bc4-d2f318ad2ada"
+					(reference "#PWR017")
 					(unit 1)
 				)
@@
 		(dnp no)
 		(fields_autoplaced yes)
-		(property "Reference" "U3"
+		(property "Reference" "U4"
 			(at 109.22 53.3399 0)
 			(effects
@@
 				)
 			)
+			(project ""
+				(path "/7776e3ee-622a-4a3e-a213-279f6f5df2cb/09f4a7ab-b5f1-4ef7-9bc4-d2f318ad2ada"
+					(reference "U4")
+					(unit 3)
+				)
+			)
 		)
 	)
@@
 		(dnp no)
 		(fields_autoplaced yes)
-		(property "Reference" "C21"
+		(property "Reference" "C18"
 			(at 115.57 111.7599 0)
 			(effects
@@
 				)
 			)
+			(project ""
+				(path "/7776e3ee-622a-4a3e-a213-279f6f5df2cb/09f4a7ab-b5f1-4ef7-9bc4-d2f318ad2ada"
+					(reference "C18")
+					(unit 1)
+				)
+			)
 		)
 	)
@@
 		(dnp no)
 		(fields_autoplaced yes)
-		(property "Reference" "#PWR029"
+		(property "Reference" "#PWR018"
 			(at 204.47 125.73 0)
 			(effects
@@
 				)
 			)
+			(project "mini-vehiculo-exploracion-pcb"
+				(path "/7776e3ee-622a-4a3e-a213-279f6f5df2cb/09f4a7ab-b5f1-4ef7-9bc4-d2f318ad2ada"
+					(reference "#PWR018")
+					(unit 1)
+				)
+			)
 		)
 	)
@@
 		(dnp no)
 		(fields_autoplaced yes)
-		(property "Reference" "R24"
+		(property "Reference" "R14"
 			(at 198.12 93.98 90)
 			(effects
@@
 				(path "/3cb3b833-c38f-47b4-b7e9-f0e6337b7613/27757aec-ab0f-470c-ac2a-d85fc9232d35"
 					(reference "R24")
+					(unit 1)
+				)
+			)
+			(project "mini-vehiculo-exploracion-pcb"
+				(path "/7776e3ee-622a-4a3e-a213-279f6f5df2cb/09f4a7ab-b5f1-4ef7-9bc4-d2f318ad2ada"
+					(reference "R14")
 					(unit 1)
 				)
@@
 		(dnp no)
 		(fields_autoplaced yes)
-		(property "Reference" "U3"
+		(property "Reference" "U4"
 			(at 130.81 90.17 0)
 			(effects
@@
 				)
 			)
+			(project ""
+				(path "/7776e3ee-622a-4a3e-a213-279f6f5df2cb/09f4a7ab-b5f1-4ef7-9bc4-d2f318ad2ada"
+					(reference "U4")
+					(unit 1)
+				)
+			)
 		)
 	)
@@
 		(dnp no)
 		(fields_autoplaced yes)
-		(property "Reference" "C23"
+		(property "Reference" "C21"
 			(at 219.71 66.04 90)
 			(effects
@@
 				)
 			)
+			(project "mini-vehiculo-exploracion-pcb"
+				(path "/7776e3ee-622a-4a3e-a213-279f6f5df2cb/09f4a7ab-b5f1-4ef7-9bc4-d2f318ad2ada"
+					(reference "C21")
+					(unit 1)
+				)
+			)
 		)
 	)
@@
 		(dnp no)
 		(fields_autoplaced yes)
-		(property "Reference" "#PWR026"
+		(property "Reference" "#PWR015"
 			(at 54.61 127 0)
 			(effects
@@
 				)
 			)
+			(project ""
+				(path "/7776e3ee-622a-4a3e-a213-279f6f5df2cb/09f4a7ab-b5f1-4ef7-9bc4-d2f318ad2ada"
+					(reference "#PWR015")
+					(unit 1)
+				)
+			)
 		)
 	)
@@
 		(dnp no)
 		(fields_autoplaced yes)
-		(property "Reference" "R20"
+		(property "Reference" "R10"
 			(at 57.15 110.4899 0)
 			(effects
@@
 				)
 			)
+			(project "mini-vehiculo-exploracion-pcb"
+				(path "/7776e3ee-622a-4a3e-a213-279f6f5df2cb/09f4a7ab-b5f1-4ef7-9bc4-d2f318ad2ada"
+					(reference "R10")
+					(unit 1)
+				)
+			)
 		)
 	)
@@
 				)
 			)
+			(project "mini-vehiculo-exploracion-pcb"
+				(path "/7776e3ee-622a-4a3e-a213-279f6f5df2cb/09f4a7ab-b5f1-4ef7-9bc4-d2f318ad2ada"
+					(reference "TP2")
+					(unit 1)
+				)
+			)
 		)
 	)
@@
 				)
 			)
+			(project ""
+				(path "/7776e3ee-622a-4a3e-a213-279f6f5df2cb/09f4a7ab-b5f1-4ef7-9bc4-d2f318ad2ada"
+					(reference "TP1")
+					(unit 1)
+				)
+			)
 		)
 	)
@@
 		(dnp no)
 		(fields_autoplaced yes)
-		(property "Reference" "R4"
+		(property "Reference" "R9"
 			(at 57.15 90.1699 0)
 			(effects
@@
 				)
 			)
+			(project ""
+				(path "/7776e3ee-622a-4a3e-a213-279f6f5df2cb/09f4a7ab-b5f1-4ef7-9bc4-d2f318ad2ada"
+					(reference "R9")
+					(unit 1)
+				)
+			)
 		)
 	)
@@
 		(dnp no)
 		(fields_autoplaced yes)
-		(property "Reference" "#PWR028"
+		(property "Reference" "#PWR016"
 			(at 107.95 71.12 0)
 			(effects
@@
 				)
 			)
+			(project "mini-vehiculo-exploracion-pcb"
+				(path "/7776e3ee-622a-4a3e-a213-279f6f5df2cb/09f4a7ab-b5f1-4ef7-9bc4-d2f318ad2ada"
+					(reference "#PWR016")
+					(unit 1)
+				)
+			)
 		)
 	)
@@
 		(dnp no)
 		(fields_autoplaced yes)
-		(property "Reference" "R23"
+		(property "Reference" "R13"
 			(at 180.34 93.98 90)
 			(effects
@@
 				)
 			)
+			(project "mini-vehiculo-exploracion-pcb"
+				(path "/7776e3ee-622a-4a3e-a213-279f6f5df2cb/09f4a7ab-b5f1-4ef7-9bc4-d2f318ad2ada"
+					(reference "R13")
+					(unit 1)
+				)
+			)
 		)
 	)
@@
 				)
 			)
+			(project "mini-vehiculo-exploracion-pcb"
+				(path "/7776e3ee-622a-4a3e-a213-279f6f5df2cb/09f4a7ab-b5f1-4ef7-9bc4-d2f318ad2ada"
+					(reference "TP3")
+					(unit 1)
+				)
+			)
 		)
 	)
@@
 		(dnp no)
 		(fields_autoplaced yes)
-		(property "Reference" "C22"
+		(property "Reference" "C19"
 			(at 132.08 67.31 90)
 			(effects
@@
 				)
 			)
+			(project ""
+				(path "/7776e3ee-622a-4a3e-a213-279f6f5df2cb/09f4a7ab-b5f1-4ef7-9bc4-d2f318ad2ada"
+					(reference "C19")
+					(unit 1)
+				)
+			)
 		)
 	)
@@
 		(dnp no)
 		(fields_autoplaced yes)
-		(property "Reference" "C24"
+		(property "Reference" "C20"
 			(at 208.28 110.4899 0)
 			(effects
@@
 					(unit 1)
 				)
+			)
+			(project "mini-vehiculo-exploracion-pcb"
+				(path "/7776e3ee-622a-4a3e-a213-279f6f5df2cb/09f4a7ab-b5f1-4ef7-9bc4-d2f318ad2ada"
+					(reference "C20")
+					(unit 1)
+				)

Commit message: cambio circuito 5V pcb control
Parts:
- renumbered C18 to C21, C19 to C22, C21 to C23, C20 to C24, R10 to R20, R11 to R21, R12 to R22, R13 to R23, R14 to R24, R9 to R4, U4 to U3
Changed lines of the file:
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@@
 		(dnp no)
 		(fields_autoplaced yes)
-		(property "Reference" "R11"
+		(property "Reference" "R21"
 			(at 76.2 96.52 90)
 			(effects
@@
 				)
 			)
-			(project "mini-vehiculo-exploracion-pcb"
-				(path "/7776e3ee-622a-4a3e-a213-279f6f5df2cb/09f4a7ab-b5f1-4ef7-9bc4-d2f318ad2ada"
-					(reference "R11")
-					(unit 1)
-				)
-			)
 		)
 	)
@@
 		(dnp no)
 		(fields_autoplaced yes)
-		(property "Reference" "R12"
+		(property "Reference" "R22"
 			(at 99.06 96.52 90)
 			(effects
@@
 				(path "/3cb3b833-c38f-47b4-b7e9-f0e6337b7613/27757aec-ab0f-470c-ac2a-d85fc9232d35"
 					(reference "R22")
-					(unit 1)
-				)
-			)
-			(project "mini-vehiculo-exploracion-pcb"
-				(path "/7776e3ee-622a-4a3e-a213-279f6f5df2cb/09f4a7ab-b5f1-4ef7-9bc4-d2f318ad2ada"
-					(reference "R12")
 					(unit 1)
 				)
@@
 		(on_board yes)
 		(dnp no)
-		(property "Reference" "U4"
+		(property "Reference" "U3"
 			(at 218.44 107.95 0)
 			(effects
@@
 		(dnp no)
 		(fields_autoplaced yes)
-		(property "Reference" "#PWR017"
+		(property "Reference" "#PWR027"
 			(at 111.76 127 0)
 			(effects
@@
 				(path "/3cb3b833-c38f-47b4-b7e9-f0e6337b7613/27757aec-ab0f-470c-ac2a-d85fc9232d35"
 					(reference "#PWR027")
-					(unit 1)
-				)
-			)
-			(project "mini-vehiculo-exploracion-pcb"
-				(path "/7776e3ee-622a-4a3e-a213-279f6f5df2cb/09f4a7ab-b5f1-4ef7-9bc4-d2f318ad2ada"
-					(reference "#PWR017")
 					(unit 1)
 				)
@@
 		(dnp no)
 		(fields_autoplaced yes)
-		(property "Reference" "U4"
+		(property "Reference" "U3"
 			(at 109.22 53.3399 0)
 			(effects
@@
 		(dnp no)
 		(fields_autoplaced yes)
-		(property "Reference" "C18"
+		(property "Reference" "C21"
 			(at 115.57 111.7599 0)
 			(effects
@@
 		(dnp no)
 		(fields_autoplaced yes)
-		(property "Reference" "#PWR018"
+		(property "Reference" "#PWR029"
 			(at 204.47 125.73 0)
 			(effects
@@
 				)
 			)
-			(project "mini-vehiculo-exploracion-pcb"
-				(path "/7776e3ee-622a-4a3e-a213-279f6f5df2cb/09f4a7ab-b5f1-4ef7-9bc4-d2f318ad2ada"
-					(reference "#PWR018")
-					(unit 1)
-				)
-			)
 		)
 	)
@@
 		(dnp no)
 		(fields_autoplaced yes)
-		(property "Reference" "R14"
+		(property "Reference" "R24"
 			(at 198.12 93.98 90)
 			(effects
@@
 				(path "/3cb3b833-c38f-47b4-b7e9-f0e6337b7613/27757aec-ab0f-470c-ac2a-d85fc9232d35"
 					(reference "R24")
-					(unit 1)
-				)
-			)
-			(project "mini-vehiculo-exploracion-pcb"
-				(path "/7776e3ee-622a-4a3e-a213-279f6f5df2cb/09f4a7ab-b5f1-4ef7-9bc4-d2f318ad2ada"
-					(reference "R14")
 					(unit 1)
 				)
@@
 		(dnp no)
 		(fields_autoplaced yes)
-		(property "Reference" "U4"
+		(property "Reference" "U3"
 			(at 130.81 90.17 0)
 			(effects
@@
 		(dnp no)
 		(fields_autoplaced yes)
-		(property "Reference" "C21"
+		(property "Reference" "C23"
 			(at 219.71 66.04 90)
 			(effects
@@
 				)
 			)
-			(project "mini-vehiculo-exploracion-pcb"
-				(path "/7776e3ee-622a-4a3e-a213-279f6f5df2cb/09f4a7ab-b5f1-4ef7-9bc4-d2f318ad2ada"
-					(reference "C21")
-					(unit 1)
-				)
-			)
 		)
 	)
@@
 		(dnp no)
 		(fields_autoplaced yes)
-		(property "Reference" "#PWR015"
+		(property "Reference" "#PWR026"
 			(at 54.61 127 0)
 			(effects
@@
 		(dnp no)
 		(fields_autoplaced yes)
-		(property "Reference" "R10"
+		(property "Reference" "R20"
 			(at 57.15 110.4899 0)
 			(effects
@@
 				)
 			)
-			(project "mini-vehiculo-exploracion-pcb"
-				(path "/7776e3ee-622a-4a3e-a213-279f6f5df2cb/09f4a7ab-b5f1-4ef7-9bc4-d2f318ad2ada"
-					(reference "R10")
-					(unit 1)
-				)
-			)
 		)
 	)
@@
 				)
 			)
-			(project "mini-vehiculo-exploracion-pcb"
-				(path "/7776e3ee-622a-4a3e-a213-279f6f5df2cb/09f4a7ab-b5f1-4ef7-9bc4-d2f318ad2ada"
-					(reference "TP2")
-					(unit 1)
-				)
-			)
 		)
 	)
@@
 		(dnp no)
 		(fields_autoplaced yes)
-		(property "Reference" "R9"
+		(property "Reference" "R4"
 			(at 57.15 90.1699 0)
 			(effects
@@
 		(dnp no)
 		(fields_autoplaced yes)
-		(property "Reference" "#PWR016"
+		(property "Reference" "#PWR028"
 			(at 107.95 71.12 0)
 			(effects
@@
 				)
 			)
-			(project "mini-vehiculo-exploracion-pcb"
-				(path "/7776e3ee-622a-4a3e-a213-279f6f5df2cb/09f4a7ab-b5f1-4ef7-9bc4-d2f318ad2ada"
-					(reference "#PWR016")
-					(unit 1)
-				)
-			)
 		)
 	)
@@
 		(dnp no)
 		(fields_autoplaced yes)
-		(property "Reference" "R13"
+		(property "Reference" "R23"
 			(at 180.34 93.98 90)
 			(effects
@@
 				)
 			)
-			(project "mini-vehiculo-exploracion-pcb"
-				(path "/7776e3ee-622a-4a3e-a213-279f6f5df2cb/09f4a7ab-b5f1-4ef7-9bc4-d2f318ad2ada"
-					(reference "R13")
-					(unit 1)
-				)
-			)
 		)
 	)
@@
 				)
 			)
-			(project "mini-vehiculo-exploracion-pcb"
-				(path "/7776e3ee-622a-4a3e-a213-279f6f5df2cb/09f4a7ab-b5f1-4ef7-9bc4-d2f318ad2ada"
-					(reference "TP3")
-					(unit 1)
-				)
-			)
 		)
 	)
@@
 		(dnp no)
 		(fields_autoplaced yes)
-		(property "Reference" "C19"
+		(property "Reference" "C22"
 			(at 132.08 67.31 90)
 			(effects
@@
 		(dnp no)
 		(fields_autoplaced yes)
-		(property "Reference" "C20"
+		(property "Reference" "C24"
 			(at 208.28 110.4899 0)
 			(effects
@@
 					(unit 1)
 				)
-			)
-			(project "mini-vehiculo-exploracion-pcb"
-				(path "/7776e3ee-622a-4a3e-a213-279f6f5df2cb/09f4a7ab-b5f1-4ef7-9bc4-d2f318ad2ada"
-					(reference "C20")
-					(unit 1)
-				)

Commit message: cambios
Parts:
- renumbered C21 to C18, C22 to C19, R4 to R9, U3 to U4
Changed lines of the file:
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@@
 		(dnp no)
 		(fields_autoplaced yes)
-		(property "Reference" "R21"
+		(property "Reference" "R?"
 			(at 76.2 96.52 90)
 			(effects
@@
 				)
 			)
+			(project "drivers-mini-vehiculo-pcb"
+				(path "/7776e3ee-622a-4a3e-a213-279f6f5df2cb/09f4a7ab-b5f1-4ef7-9bc4-d2f318ad2ada"
+					(reference "R?")
+					(unit 1)
+				)
+			)
 		)
 	)
@@
 		(dnp no)
 		(fields_autoplaced yes)
-		(property "Reference" "R22"
+		(property "Reference" "R?"
 			(at 99.06 96.52 90)
 			(effects
@@
 				(path "/3cb3b833-c38f-47b4-b7e9-f0e6337b7613/27757aec-ab0f-470c-ac2a-d85fc9232d35"
 					(reference "R22")
+					(unit 1)
+				)
+			)
+			(project "drivers-mini-vehiculo-pcb"
+				(path "/7776e3ee-622a-4a3e-a213-279f6f5df2cb/09f4a7ab-b5f1-4ef7-9bc4-d2f318ad2ada"
+					(reference "R?")
 					(unit 1)
 				)
@@
 		(on_board yes)
 		(dnp no)
-		(property "Reference" "U3"
+		(property "Reference" "U4"
 			(at 218.44 107.95 0)
 			(effects
@@
 		(dnp no)
 		(fields_autoplaced yes)
-		(property "Reference" "#PWR027"
+		(property "Reference" "#PWR0103"
 			(at 111.76 127 0)
 			(effects
@@
 				(path "/3cb3b833-c38f-47b4-b7e9-f0e6337b7613/27757aec-ab0f-470c-ac2a-d85fc9232d35"
 					(reference "#PWR027")
+					(unit 1)
+				)
+			)
+			(project "drivers-mini-vehiculo-pcb"
+				(path "/7776e3ee-622a-4a3e-a213-279f6f5df2cb/09f4a7ab-b5f1-4ef7-9bc4-d2f318ad2ada"
+					(reference "#PWR0103")
 					(unit 1)
 				)
@@
 		(dnp no)
 		(fields_autoplaced yes)
-		(property "Reference" "U3"
+		(property "Reference" "U4"
 			(at 109.22 53.3399 0)
 			(effects
@@
 		(dnp no)
 		(fields_autoplaced yes)
-		(property "Reference" "C21"
+		(property "Reference" "C18"
 			(at 115.57 111.7599 0)
 			(effects
@@
 		(dnp no)
 		(fields_autoplaced yes)
-		(property "Reference" "#PWR029"
+		(property "Reference" "#PWR0101"
 			(at 204.47 125.73 0)
 			(effects
@@
 				)
 			)
+			(project "drivers-mini-vehiculo-pcb"
+				(path "/7776e3ee-622a-4a3e-a213-279f6f5df2cb/09f4a7ab-b5f1-4ef7-9bc4-d2f318ad2ada"
+					(reference "#PWR0101")
+					(unit 1)
+				)
+			)
 		)
 	)
@@
 		(dnp no)
 		(fields_autoplaced yes)
-		(property "Reference" "R24"
+		(property "Reference" "R?"
 			(at 198.12 93.98 90)
 			(effects
@@
 				(path "/3cb3b833-c38f-47b4-b7e9-f0e6337b7613/27757aec-ab0f-470c-ac2a-d85fc9232d35"
 					(reference "R24")
+					(unit 1)
+				)
+			)
+			(project "drivers-mini-vehiculo-pcb"
+				(path "/7776e3ee-622a-4a3e-a213-279f6f5df2cb/09f4a7ab-b5f1-4ef7-9bc4-d2f318ad2ada"
+					(reference "R?")
 					(unit 1)
 				)
@@
 		(dnp no)
 		(fields_autoplaced yes)
-		(property "Reference" "U3"
+		(property "Reference" "U4"
 			(at 130.81 90.17 0)
 			(effects
@@
 		(dnp no)
 		(fields_autoplaced yes)
-		(property "Reference" "C23"
+		(property "Reference" "C?"
 			(at 219.71 66.04 90)
 			(effects
@@
 				)
 			)
+			(project "drivers-mini-vehiculo-pcb"
+				(path "/7776e3ee-622a-4a3e-a213-279f6f5df2cb/09f4a7ab-b5f1-4ef7-9bc4-d2f318ad2ada"
+					(reference "C?")
+					(unit 1)
+				)
+			)
 		)
 	)
@@
 		(dnp no)
 		(fields_autoplaced yes)
-		(property "Reference" "#PWR026"
+		(property "Reference" "#PWR015"
 			(at 54.61 127 0)
 			(effects
@@
 		(dnp no)
 		(fields_autoplaced yes)
-		(property "Reference" "R20"
+		(property "Reference" "R?"
 			(at 57.15 110.4899 0)
 			(effects
@@
 				)
 			)
+			(project "drivers-mini-vehiculo-pcb"
+				(path "/7776e3ee-622a-4a3e-a213-279f6f5df2cb/09f4a7ab-b5f1-4ef7-9bc4-d2f318ad2ada"
+					(reference "R?")
+					(unit 1)
+				)
+			)
 		)
 	)
@@
 		(dnp no)
 		(fields_autoplaced yes)
-		(property "Reference" "TP2"
+		(property "Reference" "TP?"
 			(at 163.83 67.8179 0)
 			(effects
@@
 				)
 			)
+			(project "drivers-mini-vehiculo-pcb"
+				(path "/7776e3ee-622a-4a3e-a213-279f6f5df2cb/09f4a7ab-b5f1-4ef7-9bc4-d2f318ad2ada"
+					(reference "TP?")
+					(unit 1)
+				)
+			)
 		)
 	)
@@
 		(dnp no)
 		(fields_autoplaced yes)
-		(property "Reference" "R4"
+		(property "Reference" "R9"
 			(at 57.15 90.1699 0)
 			(effects
@@
 		(dnp no)
 		(fields_autoplaced yes)
-		(property "Reference" "#PWR028"
+		(property "Reference" "#PWR0102"
 			(at 107.95 71.12 0)
 			(effects
@@
 				)
 			)
+			(project "drivers-mini-vehiculo-pcb"
+				(path "/7776e3ee-622a-4a3e-a213-279f6f5df2cb/09f4a7ab-b5f1-4ef7-9bc4-d2f318ad2ada"
+					(reference "#PWR0102")
+					(unit 1)
+				)
+			)
 		)
 	)
@@
 		(dnp no)
 		(fields_autoplaced yes)
-		(property "Reference" "R23"
+		(property "Reference" "R?"
 			(at 180.34 93.98 90)
 			(effects
@@
 				)
 			)
+			(project "drivers-mini-vehiculo-pcb"
+				(path "/7776e3ee-622a-4a3e-a213-279f6f5df2cb/09f4a7ab-b5f1-4ef7-9bc4-d2f318ad2ada"
+					(reference "R?")
+					(unit 1)
+				)
+			)
 		)
 	)
@@
 		(dnp no)
 		(fields_autoplaced yes)
-		(property "Reference" "TP3"
+		(property "Reference" "TP?"
 			(at 243.84 66.5479 0)
 			(effects
@@
 				)
 			)
+			(project "drivers-mini-vehiculo-pcb"
+				(path "/7776e3ee-622a-4a3e-a213-279f6f5df2cb/09f4a7ab-b5f1-4ef7-9bc4-d2f318ad2ada"
+					(reference "TP?")
+					(unit 1)
+				)
+			)
 		)
 	)
@@
 		(dnp no)
 		(fields_autoplaced yes)
-		(property "Reference" "C22"
+		(property "Reference" "C19"
 			(at 132.08 67.31 90)
 			(effects
@@
 		(dnp no)
 		(fields_autoplaced yes)
-		(property "Reference" "C24"
+		(property "Reference" "C?"
 			(at 208.28 110.4899 0)
 			(effects
@@
 					(unit 1)
 				)
+			)
+			(project "drivers-mini-vehiculo-pcb"
+				(path "/7776e3ee-622a-4a3e-a213-279f6f5df2cb/09f4a7ab-b5f1-4ef7-9bc4-d2f318ad2ada"
+					(reference "C?")
+					(unit 1)
+				)

Commit message: changes etc
Parts:
- removed C23: 4.7u, symbol Device:C
- removed C24: 10uF, symbol Device:C
- removed R20: 10k, symbol Device:R
- removed R21: 18k, symbol Device:R
- removed R22: 20k, symbol Device:R
- removed R23: 2k, symbol Device:R
- removed R24: 2.7k, symbol Device:R
- added C20: 10uF, Capacitor_SMD:C_0805_2012Metric_Pad1.18x1.45mm_HandSolder, symbol Device:C
- added C21: 4.7u, Capacitor_SMD:C_0805_2012Metric_Pad1.18x1.45mm_HandSolder, symbol Device:C
- added R10: 10k, Resistor_SMD:R_0805_2012Metric_Pad1.20x1.40mm_HandSolder, symbol Device:R
- added R11: 18k, Resistor_SMD:R_0805_2012Metric_Pad1.20x1.40mm_HandSolder, symbol Device:R
- added R12: 20k, Resistor_SMD:R_0805_2012Metric_Pad1.20x1.40mm_HandSolder, symbol Device:R
- added R13: 2k, Resistor_SMD:R_0805_2012Metric_Pad1.20x1.40mm_HandSolder, symbol Device:R
- added R14: 2.7k, Resistor_SMD:R_0805_2012Metric_Pad1.20x1.40mm_HandSolder, symbol Device:R
- C18, C19: footprint (none) -> Capacitor_SMD:C_0805_2012Metric_Pad1.18x1.45mm_HandSolder
- R9: footprint (none) -> Resistor_SMD:R_0805_2012Metric_Pad1.20x1.40mm_HandSolder
- TP1: footprint (none) -> TestPoint:TestPoint_Pad_1.5x1.5mm
- TP2: value OP1_Out -> OP2_Out; footprint (none) -> TestPoint:TestPoint_Pad_1.5x1.5mm
- TP3: value OP2_Out -> OP1_Out; footprint (none) -> TestPoint:TestPoint_Pad_1.5x1.5mm
Connections:
- net ADC_BAT: now also TP2.1, C21.2; no longer TP3.1
- net GND: now also C20.2, R10.1
- net OP1_OUT: now also TP3.1, R13.1; no longer TP2.1
- net at C19.1: now also R11.1, R12.1
- net at R9.1, TP1.1: now also R10.2, R11.2
- net at C18.1, U4.3 (+): now also R12.2
- net at U4.5 (+): now also C20.1, R14.2
- new net: C21.1, R13.2, R14.1

Commit message: Add footprints
Parts:
- removed C20: 10uF, Capacitor_SMD:C_0805_2012Metric_Pad1.18x1.45mm_HandSolder, symbol Device:C
- removed C21: 4.7u, Capacitor_SMD:C_0805_2012Metric_Pad1.18x1.45mm_HandSolder, symbol Device:C
- removed R10: 10k, Resistor_SMD:R_0805_2012Metric_Pad1.20x1.40mm_HandSolder, symbol Device:R
- removed R11: 18k, Resistor_SMD:R_0805_2012Metric_Pad1.20x1.40mm_HandSolder, symbol Device:R
- removed R12: 20k, Resistor_SMD:R_0805_2012Metric_Pad1.20x1.40mm_HandSolder, symbol Device:R
- removed R13: 2k, Resistor_SMD:R_0805_2012Metric_Pad1.20x1.40mm_HandSolder, symbol Device:R
- removed R14: 2.7k, Resistor_SMD:R_0805_2012Metric_Pad1.20x1.40mm_HandSolder, symbol Device:R
- added C17: 10uF, Capacitor_SMD:C_0805_2012Metric_Pad1.18x1.45mm_HandSolder, symbol Device:C
- added C18: 4.7u, Capacitor_SMD:C_0805_2012Metric_Pad1.18x1.45mm_HandSolder, symbol Device:C
- added R15: 10k, Resistor_SMD:R_0805_2012Metric_Pad1.20x1.40mm_HandSolder, symbol Device:R
- added R16: 18k, Resistor_SMD:R_0805_2012Metric_Pad1.20x1.40mm_HandSolder, symbol Device:R
- added R17: 20k, Resistor_SMD:R_0805_2012Metric_Pad1.20x1.40mm_HandSolder, symbol Device:R
- added R20: 2k, Resistor_SMD:R_0805_2012Metric_Pad1.20x1.40mm_HandSolder, symbol Device:R
- added R21: 2.7k, Resistor_SMD:R_0805_2012Metric_Pad1.20x1.40mm_HandSolder, symbol Device:R
- TP2: value OP2_Out -> OP1_Out
- TP3: value OP1_Out -> OP2_Out
- renumbered C18 to C21, C19 to C22, R9 to R4, U4 to U3
Connections:
- net ADC_BAT: now also TP3.1, C18.2; no longer TP2.1
- net GND: now also C17.2, R15.1
- net OP1_OUT: now also TP2.1, R20.1; no longer TP3.1
- net at C22.1: now also R16.1, R17.1
- net at C21.1, U3.3 (+): now also R17.2
- net at U3.5 (+): now also C17.1, R21.2
- net at R4.1, TP1.1: now also R15.2, R16.2
- new net: C18.1, R20.2, R21.1

Commit message: Add footprints
Parts:
- U3: footprint (none) -> LM358AN_NOPB:DIP794W53P254L959H508Q8N
Changed lines of the file:
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@@
 			)
 		)
-		(property "Footprint" ""
+		(property "Footprint" "LM358AN_NOPB:DIP794W53P254L959H508Q8N"
 			(at 218.44 97.79 0)
 			(effects
@@
 			)
 		)
-		(property "Footprint" ""
+		(property "Footprint" "LM358AN_NOPB:DIP794W53P254L959H508Q8N"
 			(at 110.49 54.61 0)
 			(effects
@@
 			)
 		)
-		(property "Footprint" ""
+		(property "Footprint" "LM358AN_NOPB:DIP794W53P254L959H508Q8N"
 			(at 130.81 100.33 0)
 			(effects
