File: Hardware/mini-vehiculo-exploracion-pcb/battery_sensor.kicad_sch (KiCad schematic)
At the start: 14 parts, among them U4 LM358

Commit message: Add hardware to main
Parts:
- renumbered C20 to C17, C21 to C18, C18 to C21, C19 to C22, R10 to R15, R11 to R16, R12 to R17, R13 to R20, R14 to R21, R9 to R4, U4 to U3
Changed lines of the file:
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@@
 		(dnp no)
 		(fields_autoplaced yes)
-		(property "Reference" "C21"
+		(property "Reference" "C18"
 			(at 219.71 66.04 90)
 			(effects
@@
 			(project "drivers-mini-vehiculo-pcb"
 				(path "/7776e3ee-622a-4a3e-a213-279f6f5df2cb/09f4a7ab-b5f1-4ef7-9bc4-d2f318ad2ada"
-					(reference "C21")
+					(reference "C?")
 					(unit 1)
 				)
@@
 		(dnp no)
 		(fields_autoplaced yes)
-		(property "Reference" "C20"
+		(property "Reference" "C17"
 			(at 208.28 110.4899 0)
 			(effects
@@
 			(project "drivers-mini-vehiculo-pcb"
 				(path "/7776e3ee-622a-4a3e-a213-279f6f5df2cb/09f4a7ab-b5f1-4ef7-9bc4-d2f318ad2ada"
-					(reference "C20")
+					(reference "C?")
 					(unit 1)
 				)
@@
 		(dnp no)
 		(fields_autoplaced yes)
-		(property "Reference" "R10"
+		(property "Reference" "R15"
 			(at 57.15 110.4899 0)
 			(effects
@@
 			(project "drivers-mini-vehiculo-pcb"
 				(path "/7776e3ee-622a-4a3e-a213-279f6f5df2cb/09f4a7ab-b5f1-4ef7-9bc4-d2f318ad2ada"
-					(reference "R10")
+					(reference "R?")
 					(unit 1)
 				)
@@
 		(dnp no)
 		(fields_autoplaced yes)
-		(property "Reference" "R11"
+		(property "Reference" "R16"
 			(at 76.2 96.52 90)
 			(effects
@@
 			(project "drivers-mini-vehiculo-pcb"
 				(path "/7776e3ee-622a-4a3e-a213-279f6f5df2cb/09f4a7ab-b5f1-4ef7-9bc4-d2f318ad2ada"
-					(reference "R11")
+					(reference "R?")
 					(unit 1)
 				)
@@
 		(on_board yes)
 		(dnp no)
-		(property "Reference" "U4"
+		(property "Reference" "U3"
 			(at 218.44 107.95 0)
 			(effects
@@
 		(dnp no)
 		(fields_autoplaced yes)
-		(property "Reference" "#PWR0103"
+		(property "Reference" "#PWR027"
 			(at 111.76 127 0)
 			(effects
@@
 		(dnp no)
 		(fields_autoplaced yes)
-		(property "Reference" "U4"
+		(property "Reference" "U3"
 			(at 109.22 53.3399 0)
 			(effects
@@
 		(dnp no)
 		(fields_autoplaced yes)
-		(property "Reference" "C18"
+		(property "Reference" "C21"
 			(at 115.57 111.7599 0)
 			(effects
@@
 		(dnp no)
 		(fields_autoplaced yes)
-		(property "Reference" "#PWR0101"
+		(property "Reference" "#PWR029"
 			(at 204.47 125.73 0)
 			(effects
@@
 			(project "drivers-mini-vehiculo-pcb"
 				(path "/7776e3ee-622a-4a3e-a213-279f6f5df2cb/09f4a7ab-b5f1-4ef7-9bc4-d2f318ad2ada"
-					(reference "TP2")
+					(reference "TP?")
 					(unit 1)
 				)
@@
 		(dnp no)
 		(fields_autoplaced yes)
-		(property "Reference" "R13"
+		(property "Reference" "R20"
 			(at 180.34 93.98 90)
 			(effects
@@
 			(project "drivers-mini-vehiculo-pcb"
 				(path "/7776e3ee-622a-4a3e-a213-279f6f5df2cb/09f4a7ab-b5f1-4ef7-9bc4-d2f318ad2ada"
-					(reference "R13")
+					(reference "R?")
 					(unit 1)
 				)
@@
 		(dnp no)
 		(fields_autoplaced yes)
-		(property "Reference" "U4"
+		(property "Reference" "U3"
 			(at 130.81 90.17 0)
 			(effects
@@
 		(dnp no)
 		(fields_autoplaced yes)
-		(property "Reference" "#PWR015"
+		(property "Reference" "#PWR026"
 			(at 54.61 127 0)
 			(effects
@@
 		(dnp no)
 		(fields_autoplaced yes)
-		(property "Reference" "R9"
+		(property "Reference" "R4"
 			(at 57.15 90.1699 0)
 			(effects
@@
 		(dnp no)
 		(fields_autoplaced yes)
-		(property "Reference" "R12"
+		(property "Reference" "R17"
 			(at 99.06 96.52 90)
 			(effects
@@
 			(project "drivers-mini-vehiculo-pcb"
 				(path "/7776e3ee-622a-4a3e-a213-279f6f5df2cb/09f4a7ab-b5f1-4ef7-9bc4-d2f318ad2ada"
-					(reference "R12")
+					(reference "R?")
 					(unit 1)
 				)
@@
 			(project "drivers-mini-vehiculo-pcb"
 				(path "/7776e3ee-622a-4a3e-a213-279f6f5df2cb/09f4a7ab-b5f1-4ef7-9bc4-d2f318ad2ada"
-					(reference "TP3")
+					(reference "TP?")
 					(unit 1)
 				)
@@
 		(dnp no)
 		(fields_autoplaced yes)
-		(property "Reference" "R14"
+		(property "Reference" "R21"
 			(at 198.12 93.98 90)
 			(effects
@@
 			(project "drivers-mini-vehiculo-pcb"
 				(path "/7776e3ee-622a-4a3e-a213-279f6f5df2cb/09f4a7ab-b5f1-4ef7-9bc4-d2f318ad2ada"
-					(reference "R14")
+					(reference "R?")
 					(unit 1)
 				)
@@
 		(dnp no)
 		(fields_autoplaced yes)
-		(property "Reference" "#PWR0102"
+		(property "Reference" "#PWR028"
 			(at 107.95 71.12 0)
 			(effects
@@
 		(dnp no)
 		(fields_autoplaced yes)
-		(property "Reference" "C19"
+		(property "Reference" "C22"
 			(at 132.08 67.31 90)
 			(effects
