File: Hardware/mini-vehiculo-exploracion-pcb/mcu.kicad_sch (KiCad schematic)
At the start: 20 parts, among them J2 USB_C_Receptacle_USB2.0_16P

Commit message: update pcb3
Parts:
- removed J2: USB_C_Receptacle_USB2.0_16P, USB_UJ20-C-H-G-SMT-P16-TR:SAMESKY_UJ20-C-H-G-SMT-P16-TR, symbol Connector:USB_C_Receptacle_USB2.0_16P
- added J3: UJ20-C-H-G-SMT-5-P16-TR, USB_UJ20-C-H-G-SMT-P16-TR:UJ20CHGSMT5P16TR, symbol UJ20-C-H-G-SMT-5-P16-TR:UJ20-C-H-G-SMT-5-P16-TR
- D6: value GREEN -> ON
- renumbered S2 to BOOT1
Connections:
- net CC1: now also J3.A5 (CC1)
- net CC2: now also J3.B5 (CC2)
- net D+: now also J3.A6 (DP1), J3.B6 (DP2)
- net D-: now also J3.A7 (DN1), J3.B7 (DN2)
- net GND: now also J3.A1 (GND_1), J3.B1 (GND_2)
- net V_BUS: now also F1.1, J3.A4 (VBUS_1), J3.B4 (VBUS_2)
- no-connect marks 6 -> 10
Other:
- moved on the sheet: C12, CR1, D1, D6, F1, FB1, R10, R11, R18

Commit message: Reorder
Other:
- note removed: "Planilla OK"
- title: (none) -> Vehiculo de exploracion a escala
Changed lines of the file:
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@@
 	(generator_version "9.0")
 	(paper "A4")
-	(text "Planilla OK"
-		(exclude_from_sim no)
-		(at 94.488 25.146 0)
-		(effects
-			(font
-				(size 1.27 1.27)
-				(color 245 0 255 1)
-			)
-		)
-	)
-	(text "Planilla OK"
-		(exclude_from_sim no)
-		(at 133.096 84.074 0)
-		(effects
-			(font
-				(size 1.27 1.27)
-				(color 245 0 255 1)
-			)
-		)
+	(title_block
+		(title "Vehiculo de exploracion a escala")
+		(date "2026-03-28")
+		(rev "1.0")
 	)
 	(text_box "BOOT"
