File: Hardware/mini-vehiculo-exploracion-pcb/electrical_drivers.kicad_sch (KiCad schematic)
At the start: 13 parts, among them IC1 MAX8891EXK33_V+T, U3 TPS561208DDCR

Commit message: Revert "cambios"
This reverts commit 18d6c077649d06db3e4be51193d20dbced0bef3d, reversing
changes made to f53350afebab44693d0a4c4c217b64a1fc0c425b.
Parts:
- L1: footprint MLP2520S4R7MT0S1:INDC2520X100N -> (none)
Changed lines of the file:
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@@
 			)
 		)
-		(property "Footprint" "MLP2520S4R7MT0S1:INDC2520X100N"
+		(property "Footprint" ""
 			(at 106.68 39.37 0)
 			(effects

Commit message: Add netclassses, mounting holes and terminal block
Parts:
- L1: footprint (none) -> MLP2520S4R7MT0S1:INDC2520X100N
Changed lines of the file:
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@@
 			)
 		)
-		(property "Footprint" ""
+		(property "Footprint" "MLP2520S4R7MT0S1:INDC2520X100N"
 			(at 106.68 39.37 0)
 			(effects

Commit message: cambios rama de drivers
Parts:
- removed L1: 4,7u, MLP2520S4R7MT0S1:INDC2520X100N, symbol Device:L
- added L1: MLP2520S4R7MT0S1, INDC2520X100N, symbol MLP2520S4R7MT0S1:MLP2520S4R7MT0S1
Connections:
- net +5V: now also L1.2
- net at C14.2, U3.2 (SW): now also L1.1
Other:
- moved on the sheet: C15, R7, R8

Commit message: cambio de fusible
Parts:
- removed F1: SF-1206SA1500R-2, SF-1206SA1500R-2:SF1206SA1500R2, symbol SF-1206SA1500R-2:SF-1206SA1500R-2
- added F1: SF-1206SA1500W-2, FUSC3217X123N, symbol SF-1206SA1500W-2:SF-1206SA1500W-2
Connections:
- net V_BAT: now also F1.1
- net at D2.1 (A_1), D2.2 (A_2): now also F1.2
