File: Hardware/mini-vehiculo-exploracion-pcb/drivers-mini-vehiculo-pcb.kicad_pcb (KiCad board)
At the start: 2 copper layers, 70.3 x 98.5 mm, 56 parts, among them IC1 MAX8891EXK33_V+T, J1 Conn_01x08_Pin_drv, J2 Conn_01x02_Pin_drv, J4 Motor1_Terminal, J4 Motor2_Terminal, J5 Battery_Terminal_01x02, U1 DRV8873HPWPRQ1, U2 DRV8873HPWPRQ1, U3 TPS561208DDCR, U4 LM358

Commit message: reduced vias quantity
Routing:
- net GND: vias 322 -> 120
Other:
- board text added: "MOTOR 1"
- board text added: "MOTOR 2"

Commit message: added logo
Parts:
- added G***: LOGO, logo:luna1, F.Cu at (83.5, 120.0)
- added G***: LOGO, logo:rover, F.Cu at (74.0, 123.7)
